File: KiCad/RPNCalcProject/RPNCalcProject.kicad_sch (KiCad schematic)
At the start: 103 parts, among them J1 Barrel_Jack_Switch, SW1 RCL, SW10 IMAGINARY, SW11 NUM_7, SW12 NUM_4, SW13 NUM_1, SW14 NUM_0, SW15 SWAP, SW16 TAN, SW17 NEGATE, SW18 NUM_8, SW19 NUM_5, SW2 SIN, SW20 NUM_2, SW21 DECIMAL, SW22 ARROW_LEFT, SW23 POWER, SW24 ENG_NOTATION, SW25 NUM_9, SW26 NUM_6, SW27 NUM_3, SW28 FACTORIAL, SW29 ARROW_RIGHT, SW3 ENTER, SW30 INVERSE, SW31 BACKSPACE, SW32 DIVIDE, SW33 MULTIPLY, SW34 SUBTRACT, SW35 ADD, SW4 SYMBOLS, SW5 SWITCH, SW6 CLEAR, SW7 OFF/ON, SW8 STACK_DOWN, SW9 COS, U1 MSP430G2553IPW20, U2 MCP23017_SO, U3 74HC595, U4 MIC5365-3.3YC5

Commit message: Updated KiCad schematic
Connections:
- net P1.1: now reaches DS2.3 (VO)
- net P1.1: now also U1.3 (UCA0RXD/UCA0SOMI/TA0.0/CA1/A1/P1.1)
- no-connect marks 17 -> 16
Other:
- note removed: "Put potentiometer here"
- moved on the sheet: C1, C2, U4
Changed lines of the file:
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@@
 		)
 	)
-	(text "Put potentiometer here\n"
-		(exclude_from_sim no)
-		(at 325.882 119.38 0)
-		(effects
-			(font
-				(size 1.27 1.27)
-			)
-		)
-	)
 	(text "MSP430G2553 MCU\n"
 		(exclude_from_sim no)
@@
 	)
 	(junction
-		(at 62.23 38.1)
+		(at 64.77 38.1)
 		(diameter 0)
 		(color 0 0 0 0)
 	)
 	(junction
-		(at 90.17 38.1)
+		(at 92.71 38.1)
 		(diameter 0)
 		(color 0 0 0 0)
 	)
 	(junction
-		(at 50.8 38.1)
+		(at 53.34 38.1)
 		(diameter 0)
 		(color 0 0 0 0)
@@
 	)
 	(junction
-		(at 76.2 48.26)
+		(at 78.74 48.26)
 		(diameter 0)
 		(color 0 0 0 0)
@@
 	)
 	(no_connect
-		(at 245.11 41.91)
-	)
-	(no_connect
 		(at 245.11 52.07)
 	)
@@
 	(wire
 		(pts
-			(xy 50.8 38.1) (xy 62.23 38.1)
+			(xy 53.34 38.1) (xy 64.77 38.1)
 		)
 		(stroke
@@
 	(wire
 		(pts
-			(xy 62.23 48.26) (xy 76.2 48.26)
+			(xy 64.77 48.26) (xy 78.74 48.26)
 		)
 		(stroke
@@
 	(wire
 		(pts
-			(xy 86.36 38.1) (xy 90.17 38.1)
+			(xy 88.9 38.1) (xy 92.71 38.1)
 		)
 		(stroke
@@
 	(wire
 		(pts
-			(xy 66.04 43.18) (xy 50.8 43.18)
+			(xy 68.58 43.18) (xy 53.34 43.18)
 		)
 		(stroke
@@
 	(wire
 		(pts
-			(xy 76.2 48.26) (xy 90.17 48.26)
+			(xy 78.74 48.26) (xy 92.71 48.26)
 		)
 		(stroke
@@
 	(wire
 		(pts
-			(xy 95.25 38.1) (xy 95.25 35.56)
+			(xy 40.64 38.1) (xy 53.34 38.1)
 		)
 		(stroke
@@
 	(wire
 		(pts
-			(xy 62.23 45.72) (xy 62.23 48.26)
+			(xy 97.79 38.1) (xy 97.79 35.56)
 		)
 		(stroke
@@
 	(wire
 		(pts
-			(xy 90.17 38.1) (xy 95.25 38.1)
+			(xy 64.77 45.72) (xy 64.77 48.26)
 		)
 		(stroke
@@
 	(wire
 		(pts
-			(xy 76.2 48.26) (xy 76.2 49.53)
+			(xy 92.71 38.1) (xy 97.79 38.1)
 		)
 		(stroke
@@
 	(wire
 		(pts
-			(xy 40.64 43.18) (xy 40.64 48.26)
+			(xy 78.74 48.26) (xy 78.74 49.53)
 		)
 		(stroke
@@
 	(wire
 		(pts
-			(xy 255.27 57.15) (xy 245.11 57.15)
+			(xy 40.64 43.18) (xy 40.64 48.26)
 		)
 		(stroke
@@
 	(wire
 		(pts
-			(xy 259.08 57.15) (xy 255.27 57.15)
+			(xy 255.27 57.15) (xy 245.11 57.15)
 		)
 		(stroke
@@
 	(wire
 		(pts
-			(xy 40.64 38.1) (xy 50.8 38.1)
+			(xy 259.08 57.15) (xy 255.27 57.15)
 		)
 		(stroke
@@
 	(wire
 		(pts
-			(xy 62.23 38.1) (xy 66.04 38.1)
+			(xy 64.77 38.1) (xy 68.58 38.1)
 		)
 		(stroke
@@
 	(wire
 		(pts
-			(xy 90.17 45.72) (xy 90.17 48.26)
+			(xy 92.71 45.72) (xy 92.71 48.26)
 		)
 		(stroke
@@
 	(wire
 		(pts
-			(xy 50.8 43.18) (xy 50.8 38.1)
+			(xy 53.34 43.18) (xy 53.34 38.1)
 		)
 		(stroke
@@
 		)
 	)
+	(global_label "P1.1"
+		(shape output)
+		(at 245.11 41.91 0)
+		(fields_autoplaced yes)
+		(effects
+			(font
+				(size 1.27 1.27)
+			)
+			(justify left)
+		)
+		(property "Intersheetrefs" "${INTERSHEET_REFS}"
+			(at 252.389 41.91 0)
+			(effects
+				(font
+					(size 1.27 1.27)
+				)
+				(justify left)
+				(hide yes)
+			)
+		)
+	)
 	(global_label "LCD_D5"
 		(shape input)
@@
 		)
 	)
+	(global_label "P1.1"
+		(shape input)
+		(at 313.69 119.38 0)
+		(fields_autoplaced yes)
+		(effects
+			(font
+				(size 1.27 1.27)
+			)
+			(justify left)
+		)
+		(property "Intersheetrefs" "${INTERSHEET_REFS}"
+			(at 320.969 119.38 0)
+			(effects
+				(font
+					(size 1.27 1.27)
+				)
+				(justify left)
+				(hide yes)
+			)
+		)
+	)
 	(global_label "GPA2"
 		(shape output)
@@
 	(symbol
 		(lib_id "power:GND")
-		(at 76.2 49.53 0)
+		(at 78.74 49.53 0)
 		(unit 1)
 		(exclude_from_sim no)
@@
 		(fields_autoplaced yes)
 		(property "Reference" "#PWR021"
-			(at 76.2 55.88 0)
+			(at 78.74 55.88 0)
 			(effects
 				(font
@@
 		)
 		(property "Value" "GND"
-			(at 76.2 54.61 0)
+			(at 78.74 54.61 0)
 			(effects
 				(font
@@
 		)
 		(property "Footprint" ""
-			(at 76.2 49.53 0)
+			(at 78.74 49.53 0)
 			(effects
 				(font
@@
 		)
 		(property "Datasheet" ""
-			(at 76.2 49.53 0)
+			(at 78.74 49.53 0)
 			(effects
 				(font
@@
 		)
 		(property "Description" "Power symbol creates a global label with name \"GND\" , ground"
-			(at 76.2 49.53 0)
+			(at 78.74 49.53 0)
 			(effects
 				(font
@@
 	(symbol
 		(lib_id "power:+3.3V")
-		(at 95.25 35.56 0)
+		(at 97.79 35.56 0)
 		(unit 1)
 		(exclude_from_sim no)
@@
 		(fields_autoplaced yes)
 		(property "Reference" "#PWR022"
-			(at 95.25 39.37 0)
+			(at 97.79 39.37 0)
 			(effects
 				(font
@@
 		)
 		(property "Value" "+3.3V"
-			(at 95.25 30.48 0)
+			(at 97.79 30.48 0)
 			(effects
 				(font
@@
 		)
 		(property "Footprint" ""
-			(at 95.25 35.56 0)
+			(at 97.79 35.56 0)
 			(effects
 				(font
@@
 		)
 		(property "Datasheet" ""
-			(at 95.25 35.56 0)
+			(at 97.79 35.56 0)
 			(effects
 				(font
@@
 		)
 		(property "Description" "Power symbol creates a global label with name \"+3.3V\""
-			(at 95.25 35.56 0)
+			(at 97.79 35.56 0)
 			(effects
 				(font
@@
 	(symbol
 		(lib_id "Regulator_Linear:MIC5365-3.3YC5")
-		(at 76.2 40.64 0)
+		(at 78.74 40.64 0)
 		(unit 1)
 		(exclude_from_sim no)
@@
 		(fields_autoplaced yes)
 		(property "Reference" "U4"
-			(at 76.2 30.48 0)
+			(at 78.74 30.48 0)
 			(effects
 				(font
@@
 		)
 		(property "Value" "MIC5365-3.3YC5"
-			(at 76.2 33.02 0)
+			(at 78.74 33.02 0)
 			(effects
 				(font
@@
 		)
 		(property "Footprint" "Package_TO_SOT_SMD:SOT-353_SC-70-5"
-			(at 76.2 29.21 0)
+			(at 78.74 29.21 0)
 			(effects
 				(font
@@
 		)
 		(property "Datasheet" "https://ww1.microchip.com/downloads/aemDocuments/documents/APID/ProductDocuments/DataSheets/MIC5365-6-High-Performance-Single-150mA-LDO-DS20006605A.pdf"
-			(at 76.2 31.75 0)
+			(at 78.74 31.75 0)
 			(effects
 				(font
@@
 		)
 		(property "Description" "150mA Low-dropout Voltage Regulator, Vout 3.3V, Vin up to 5.5V, SC-70-5"
-			(at 76.2 26.67 0)
+			(at 78.74 26.67 0)
 			(effects
 				(font
@@
 	(symbol
 		(lib_id "Device:C")
-		(at 90.17 41.91 0)
+		(at 92.71 41.91 0)
 		(unit 1)
 		(exclude_from_sim no)
@@
 		(dnp no)
 		(property "Reference" "C2"
-			(at 87.376 39.878 0)
+			(at 89.916 39.878 0)
 			(effects
 				(font
@@
 		)
 		(property "Value" "1uF"
-			(at 90.678 39.878 0)
+			(at 93.218 39.878 0)
 			(effects
 				(font
@@
 		)
 		(property "Footprint" "Capacitor_SMD:C_0201_0603Metric_Pad0.64x0.40mm_HandSolder"
-			(at 91.1352 45.72 0)
+			(at 93.6752 45.72 0)
 			(effects
 				(font
@@
 		)
 		(property "Datasheet" "~"
-			(at 90.17 41.91 0)
+			(at 92.71 41.91 0)
 			(effects
 				(font
@@
 		)
 		(property "Description" "Unpolarized capacitor"
-			(at 90.17 41.91 0)
+			(at 92.71 41.91 0)
 			(effects
 				(font
@@
 	(symbol
 		(lib_id "Device:C")
-		(at 62.23 41.91 0)
+		(at 64.77 41.91 0)
 		(unit 1)
 		(exclude_from_sim no)
@@
 		(dnp no)
 		(property "Reference" "C1"
-			(at 59.436 39.878 0)
+			(at 61.976 39.878 0)
 			(effects
 				(font
@@
 		)
 		(property "Value" "1uF"
-			(at 62.738 39.878 0)
+			(at 65.278 39.878 0)
 			(effects
 				(font
@@
 		)
 		(property "Footprint" "Capacitor_SMD:C_0201_0603Metric_Pad0.64x0.40mm_HandSolder"
-			(at 63.1952 45.72 0)
+			(at 65.7352 45.72 0)
 			(effects
 				(font
@@
 		)
 		(property "Datasheet" "~"
-			(at 62.23 41.91 0)
+			(at 64.77 41.91 0)
 			(effects
 				(font
@@
 		)
 		(property "Description" "Unpolarized capacitor"
-			(at 62.23 41.91 0)
+			(at 64.77 41.91 0)
 			(effects
 				(font
