File: KiCad/RPNCalcProject/RPNCalcProject.kicad_pcb (KiCad board)
At the start: 2 copper layers, 81 x 127 mm, 103 parts, among them J1 Barrel_Jack_Switch, SW1 RCL, SW10 IMAGINARY, SW11 NUM_7, SW12 NUM_4, SW13 NUM_1, SW14 NUM_0, SW15 SWAP, SW16 TAN, SW17 NEGATE, SW18 NUM_8, SW19 NUM_5, SW2 SIN, SW20 NUM_2, SW21 DECIMAL, SW22 ARROW_LEFT, SW23 POWER, SW24 ENG_NOTATION, SW25 NUM_9, SW26 NUM_6, SW27 NUM_3, SW28 FACTORIAL, SW29 ARROW_RIGHT, SW3 ENTER, SW30 INVERSE, SW31 BACKSPACE, SW32 DIVIDE, SW33 MULTIPLY, SW34 SUBTRACT, SW35 ADD, SW4 SYMBOLS, SW5 SWITCH, SW6 CLEAR, SW7 OFF/ON, SW8 STACK_DOWN, SW9 COS, U1 MSP430G2553IPW20, U2 MCP23017_SO, U3 74HC595, U4 MIC5365-3.3YC5

Commit message: Updated KiCad schematic
Parts:
- moved U1 30.4 mm to (144.6, 53.7), turned to -90 degrees
- moved TP6 25.8 mm to (152.3, 50.3)
- moved U3 24.6 mm to (175.0, 46.5), turned to -90 degrees
- moved TP7 22.1 mm to (157.3, 50.3)
- moved TP18 19.3 mm to (162.3, 50.3)
- moved TP17 18.5 mm to (166.8, 50.3)
- moved TP16 16.1 mm to (171.3, 53.8)
- moved TP5 13.6 mm to (155.3, 68.3)
- moved TP4 8.48 mm to (160.3, 68.3)
- moved U2 6.53 mm to (186.0, 59.5), turned to 90 degrees
- moved R1 5.43 mm to (159.2, 64.8), turned to 180 degrees
- moved TP1 3.04 mm to (187.0, 39.0)
- moved R2 3.04 mm to (154.4, 64.8), turned to 180 degrees
- moved TP19 2.83 mm to (164.8, 65.3)
- moved TP20 1.12 mm to (194.5, 71.0)
Connections:
- DS2 pad 3: unconnected-(DS2-VO-Pad3) -> P1.1
- U1 pad 3: unconnected-(U1-UCA0RXD/UCA0SOMI/TA0.0/CA1/A1/P1.1-Pad3) -> P1.1
Routing:
- net +5V: track 0.00 -> 124.6 mm, vias 0 -> 2
- net GPB6: track 62.6 -> 186.0 mm
- net GPB5: track 62.4 -> 169.2 mm
- net GPB4: track 62.6 -> 154.6 mm
- net +3.3V: track 0.00 -> 88.7 mm, vias 0 -> 6
- net GPB3: track 62.6 -> 139.6 mm
- net GND: track 0.00 -> 74.3 mm, vias 0 -> 5
- net GPA0: track 77.0 -> 141.8 mm, vias 0 -> 1
- net GPB2: track 62.4 -> 124.4 mm
- net GPA3: track 64.8 -> 121.2 mm, vias 0 -> 1
- net GPA4: track 81.3 -> 131.7 mm, vias 0 -> 1
- net GPA1: track 81.5 -> 128.0 mm, vias 0 -> 1
- net P2.2: track 0.00 -> 38.0 mm
- net GPA2: track 81.1 -> 118.2 mm, vias 0 -> 1
- net P1.7: track 0.00 -> 33.3 mm, vias 0 -> 2
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